File: PCB/myMacropad.kicad_pcb (KiCad board)
At the start: 2 copper layers, 63 x 78 mm, 21 parts, among them SW1 SW_Push, SW10 RotaryEncoder_Switch, SW2 SW_Push, SW3 SW_Push, SW4 SW_Push, SW5 SW_Push, SW6 SW_Push, SW7 SW_Push, SW8 SW_Push, SW9 SW_Push, U1 MOUDLE-SEEEDUINO-XIAO, U2 ER_OLEDM0.91_1x-I2C

Commit message: add updated files (again) via upload
Parts:
- moved D1 11.4 mm to (64.1, 67.2), turned to 180 degrees
Routing:
- net Net-(D1-A): track 13.9 -> 26.5 mm, vias 0 -> 2
- net Row 1: track 46.7 -> 49.5 mm
Changed lines of the file:
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@@
 	(footprint "Diode_THT:D_DO-35_SOD27_P7.62mm_Horizontal"
 		(layer "B.Cu")
-		(at 53.61 62.81 90)
+		(at 64.06 67.25 180)
 		(descr "Diode, DO-35_SOD27 series, Axial, Horizontal, pin pitch=7.62mm, length*diameter=4*2mm^2, http://www.diodes.com/_files/packages/DO-35.pdf")
 		(tags "Diode DO-35_SOD27 series Axial Horizontal pin pitch 7.62mm  length 4mm diameter 2mm")
 		(property "Reference" "D1"
-			(at 3.81 2.12 90)
+			(at 3.81 2.12 0)
 			(layer "B.SilkS")
 			(effects
@@
 		)
 		(property "Value" "D"
-			(at 3.81 -2.12 90)
+			(at 3.81 -2.12 0)
 			(layer "B.Fab")
 			(effects
@@
 		)
 		(property "Datasheet" ""
-			(at 0 0 90)
+			(at 0 0 0)
 			(layer "B.Fab")
 			(hide yes)
@@
 		)
 		(property "Description" "Diode"
-			(at 0 0 90)
+			(at 0 0 0)
 			(layer "B.Fab")
 			(hide yes)
@@
 		)
 		(property "KiLib_Generator" "diode/THT"
-			(at 0 0 90)
+			(at 0 0 0)
 			(layer "B.SilkS")
 			(hide yes)
@@
 		)
 		(property "Sim.Device" "D"
-			(at 0 0 270)
+			(at 0 0 0)
 			(unlocked yes)
 			(layer "B.Fab")
@@
 		)
 		(property "Sim.Pins" "1=K 2=A"
-			(at 0 0 270)
+			(at 0 0 0)
 			(unlocked yes)
 			(layer "B.Fab")
@@
 		)
 		(fp_line
-			(start 1.04 0)
-			(end 1.689999 0)
+			(start 2.53 1.12)
+			(end 2.53 -1.12)
 			(stroke
 				(width 0.12)
@@
 		)
 		(fp_line
-			(start 2.53 1.12)
-			(end 2.53 -1.12)
+			(start 2.41 1.12)
+			(end 2.41 -1.12)
 			(stroke
 				(width 0.12)
@@
 		)
 		(fp_line
-			(start 2.41 1.12)
-			(end 2.41 -1.12)
+			(start 2.29 1.12)
+			(end 2.29 -1.12)
 			(stroke
 				(width 0.12)
@@
 		)
 		(fp_line
-			(start 2.29 1.12)
-			(end 2.29 -1.12)
+			(start 1.04 0)
+			(end 1.689999 0)
 			(stroke
 				(width 0.12)
@@
 		)
 		(fp_line
-			(start 0 0)
-			(end 1.81 0)
+			(start 2.51 1)
+			(end 2.51 -1)
 			(stroke
 				(width 0.1)
@@
 		)
 		(fp_line
-			(start 2.51 1)
-			(end 2.51 -1)
+			(start 2.41 1)
+			(end 2.41 -1)
 			(stroke
 				(width 0.1)
@@
 		)
 		(fp_line
-			(start 2.41 1)
-			(end 2.41 -1)
+			(start 2.31 1)
+			(end 2.31 -1)
 			(stroke
 				(width 0.1)
@@
 		)
 		(fp_line
-			(start 2.31 1)
-			(end 2.31 -1)
+			(start 0 0)
+			(end 1.81 0)
 			(stroke
 				(width 0.1)
@@
 		)
 		(fp_text user "K"
-			(at 0 1.8 90)
+			(at 0 1.8 0)
 			(layer "B.SilkS")
 			(effects
@@
 		)
 		(fp_text user "${REFERENCE}"
-			(at 3.81 0 90)
+			(at 3.81 0 0)
 			(layer "B.Fab")
 			(effects
@@
 		)
 		(fp_text user "K"
-			(at 0 1.8 90)
+			(at 0 1.8 0)
 			(layer "B.Fab")
 			(effects
@@
 		)
 		(pad "1" thru_hole roundrect
-			(at 0 0 90)
+			(at 0 0 180)
 			(size 1.6 1.6)
 			(drill 0.8)
@@
 		)
 		(pad "2" thru_hole circle
-			(at 7.62 0 90)
+			(at 7.62 0 180)
 			(size 1.6 1.6)
 			(drill 0.8)
@@
 	)
 	(segment
-		(start 40.24 56.46)
+		(start 52.34 56.46)
+		(end 40.24 56.46)
+		(width 0.2)
+		(layer "F.Cu")
+		(net "Net-(D1-A)")
+	)
+	(segment
+		(start 54.5 56.5)
+		(end 52.38 56.5)
+		(width 0.2)
+		(layer "F.Cu")
+		(net "Net-(D1-A)")
+	)
+	(segment
+		(start 52.38 56.5)
 		(end 52.34 56.46)
 		(width 0.2)
@@
 	)
 	(segment
-		(start 52.34 56.46)
-		(end 53.61 55.19)
+		(start 55.25 67.25)
+		(end 54.5 66.5)
 		(width 0.2)
 		(layer "F.Cu")
@@
 	)
 	(segment
+		(start 56.44 67.25)
+		(end 55.25 67.25)
+		(width 0.2)
+		(layer "F.Cu")
+		(net "Net-(D1-A)")
+	)
+	(via
+		(at 54.5 56.5)
+		(size 0.6)
+		(drill 0.3)
+		(layers "F.Cu" "B.Cu")
+		(net "Net-(D1-A)")
+	)
+	(via
+		(at 54.5 66.5)
+		(size 0.6)
+		(drill 0.3)
+		(layers "F.Cu" "B.Cu")
+		(net "Net-(D1-A)")
+	)
+	(segment
+		(start 54.5 66.5)
+		(end 54.5 56.5)
+		(width 0.2)
+		(layer "B.Cu")
+		(net "Net-(D1-A)")
+	)
+	(segment
 		(start 41.51 66.625)
 		(end 37.58 62.695)
@@
 	)
 	(segment
-		(start 53.61 62.81)
-		(end 50.405 62.81)
+		(start 72.61 62.62)
+		(end 68.69 62.62)
+		(width 0.2)
+		(layer "F.Cu")
+		(net "Row 1")
+	)
+	(segment
+		(start 68.69 62.62)
+		(end 64.06 67.25)
+		(width 0.2)
+		(layer "F.Cu")
+		(net "Row 1")
+	)
+	(segment
+		(start 91.61 62.62)
+		(end 72.61 62.62)
 		(width 0.2)
 		(layer "F.Cu")
@@
 	)
 	(segment
-		(start 53.61 62.81)
-		(end 91.42 62.81)
+		(start 63 65)
+		(end 48.215 65)
 		(width 0.2)
 		(layer "F.Cu")
@@
 	)
 	(segment
-		(start 50.405 62.81)
+		(start 48.215 65)
 		(end 46.59 66.625)
 		(width 0.2)
 		(layer "F.Cu")
+		(net "Row 1")
+	)
+	(segment
+		(start 64.06 66.06)
+		(end 63 65)
+		(width 0.2)
+		(layer "F.Cu")
+		(net "Row 1")
+	)
+	(segment
+		(start 64.06 67.25)
+		(end 64.06 66.06)
+		(width 0.2)
+		(layer "F.Cu")
